File: ADC/RPi_Extension_adc.brd (EAGLE design)
At the start: 63 x 50 mm, 39 parts, among them U1 74AHC1G04GW/T1, U2 ADR423ARZ, U3 AD7616BSTZ

Commit message: updated pcbs
Parts:
- C13, C15, C16: value (none) -> 0.1u
- C14, C17: value (none) -> 10u
- R1, R3, R5: value (none) -> 10k
- moved C11 5.10 mm to (43.6, 31.9)
- moved C10 3.25 mm to (48.1, 31.9)
- moved C9 3.16 mm to (50.8, 21.1)
Routing:
- net N$2: track 5.29 -> 2.05 mm
Changed lines of the file:
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@@
 <attribute name="VENDOR" value="Vendor" x="12.35" y="5.05" size="1.778" layer="27" display="off"/>
 </element>
-<element name="C13" library="rcl" package="C0603" value="" x="6.7" y="4.85" rot="R270"/>
-<element name="C14" library="rcl" package="C1206" value="" x="3.9" y="4.3" rot="R270"/>
-<element name="C15" library="rcl" package="C0603" value="" x="17.55" y="3.6" rot="R270"/>
-<element name="C16" library="rcl" package="C0603" value="" x="16.7" y="11.45" rot="R180"/>
-<element name="C17" library="rcl" package="C1206" value="" x="16.15" y="9" rot="R180"/>
+<element name="C13" library="rcl" package="C0603" value="0.1u" x="6.7" y="4.85" rot="R270"/>
+<element name="C14" library="rcl" package="C1206" value="10u" x="3.9" y="4.3" rot="R270"/>
+<element name="C15" library="rcl" package="C0603" value="0.1u" x="17.55" y="3.6" rot="R270"/>
+<element name="C16" library="rcl" package="C0603" value="0.1u" x="16.7" y="11.45" rot="R180"/>
+<element name="C17" library="rcl" package="C1206" value="10u" x="16.15" y="9" rot="R180"/>
 <element name="SV5" library="con-lsta" package="FE20-2" value="" x="28.6" y="41.6" rot="MR180">
 <attribute name="MF" value="" x="28.6" y="41.6" size="1.778" layer="28" rot="MR180" display="off"/>
@@
 <element name="C7" library="rcl" package="C0603" value="0.1u" x="47.75" y="21.75" rot="MR180"/>
 <element name="C8" library="rcl" package="C0603" value="10u" x="47.75" y="19.15" rot="MR180"/>
-<element name="C9" library="rcl" package="C0603" value="10u" x="53.95" y="20.85" rot="R180"/>
-<element name="C10" library="rcl" package="C0603" value="0.1u" x="51.35" y="31.85" rot="R90"/>
-<element name="C11" library="rcl" package="C0603" value="10u" x="48.75" y="31.85" rot="R90"/>
+<element name="C9" library="rcl" package="C0603" value="10u" x="50.8" y="21.1" rot="R180"/>
+<element name="C10" library="rcl" package="C0603" value="0.1u" x="48.1" y="31.85" rot="R90"/>
+<element name="C11" library="rcl" package="C0603" value="10u" x="43.65" y="31.85" rot="R90"/>
 <element name="C12" library="rcl" package="C0603" value="0.1u" x="38.35" y="23.15" rot="MR180"/>
 <element name="C18" library="rcl" package="C0603" value="10u" x="38.35" y="20.05" rot="MR180"/>
 <element name="C19" library="rcl" package="C0603" value="10u" x="29.45" y="20.05" rot="MR0"/>
 <element name="C20" library="rcl" package="C0603" value="0.1u" x="29.45" y="23.55" rot="MR0"/>
-<element name="R1" library="resistor" package="R0603" value="" x="53.95" y="27.15"/>
-<element name="R3" library="resistor" package="R0603" value="" x="53.95" y="25.05"/>
+<element name="R1" library="resistor" package="R0603" value="10k" x="53.95" y="27.15"/>
+<element name="R3" library="resistor" package="R0603" value="10k" x="53.95" y="25.05"/>
 <element name="C21" library="rcl" package="C0603" value="0.1u" x="53.95" y="22.95" rot="R180"/>
-<element name="R5" library="resistor" package="R0603" value="" x="18.4" y="13.85" rot="R180"/>
+<element name="R5" library="resistor" package="R0603" value="10k" x="18.4" y="13.85" rot="R180"/>
 <element name="U1" library="74AHC1G04GW" package="SOT65P210X110-5N" value="74AHC1G04GW/T1" x="24.7" y="28.6">
 <attribute name="PACKAGE" value="SOT353-1-5" x="24.7" y="28.6" size="1.778" layer="27" display="off"/>
@@
 <contactref element="R3" pad="2"/>
 <wire x1="41.276" y1="28.421" x2="41.275" y2="28.42" width="0.4064" layer="1"/>
-<wire x1="48.75" y1="31" x2="51.35" y2="31" width="0.4064" layer="1"/>
-<wire x1="51.35" y1="31" x2="54.036784375" y2="31" width="0.4064" layer="1"/>
+<wire x1="43.65" y1="31" x2="48.1" y2="31" width="0.4064" layer="1"/>
+<wire x1="48.1" y1="31" x2="54.036784375" y2="31" width="0.4064" layer="1"/>
 <wire x1="54.036784375" y1="31" x2="54.8" y2="30.236784375" width="0.4064" layer="1"/>
 <wire x1="54.8" y1="30.236784375" x2="54.8" y2="27.15" width="0.4064" layer="1"/>
@@
 <wire x1="41.275" y1="28.42" x2="41.275" y2="30.181084375" width="0.4064" layer="1"/>
 <wire x1="41.275" y1="30.181084375" x2="42.093915625" y2="31" width="0.4064" layer="1"/>
-<wire x1="42.093915625" y1="31" x2="48.75" y2="31" width="0.4064" layer="1"/>
+<wire x1="42.093915625" y1="31" x2="43.65" y2="31" width="0.4064" layer="1"/>
 <via x="41.25" y="25.8" extent="1-16" drill="0.7"/>
 <wire x1="6.27" y1="25.8" x2="5.82" y2="25.35" width="0.4064" layer="16"/>
@@
 <contactref element="C9" pad="2"/>
 <contactref element="U3" pad="31"/>
-<wire x1="47.92" y1="21.125" x2="50.575" y2="21.125" width="0.4064" layer="1"/>
-<wire x1="53.1" y1="20.85" x2="50.85" y2="20.85" width="0.4064" layer="1"/>
-<wire x1="50.85" y1="20.85" x2="50.575" y2="21.125" width="0.4064" layer="1"/>
+<wire x1="47.92" y1="21.125" x2="49.95" y2="21.125" width="0.4064" layer="1"/>
+<wire x1="49.95" y1="21.125" x2="49.95" y2="21.1" width="0.4064" layer="1"/>
 </signal>
 <signal name="N$4">

Commit message: update
Connections:
- net CONVST: now also SV5.16; no longer SV5.18
Changed lines of the file:
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@@
 </signal>
 <signal name="CONVST">
-<contactref element="SV5" pad="18"/>
-<wire x1="24.79" y1="42.87" x2="24.79" y2="42.79" width="0.4064" layer="16"/>
-<wire x1="24.79" y1="42.79" x2="23.5" y2="41.5" width="0.4064" layer="16"/>
 <via x="21.6" y="35.95" extent="1-16" drill="0.7"/>
 <wire x1="21.6" y1="35.95" x2="21.6" y2="29.5" width="0.4064" layer="1"/>
 <wire x1="23.5" y1="37.85" x2="21.6" y2="35.95" width="0.4064" layer="16"/>
-<wire x1="23.5" y1="41.5" x2="23.5" y2="37.85" width="0.4064" layer="16"/>
+<wire x1="23.5" y1="41.62" x2="23.5" y2="37.85" width="0.4064" layer="16"/>
 <contactref element="U1" pad="2"/>
 <wire x1="21.6" y1="29.5" x2="22.5" y2="28.6" width="0.4064" layer="1"/>
 <wire x1="22.5" y1="28.6" x2="23.7348" y2="28.6" width="0.4064" layer="1"/>
+<contactref element="SV5" pad="16"/>
+<wire x1="23.5" y1="41.62" x2="22.25" y2="42.87" width="0.4064" layer="16"/>
 </signal>
 <signal name="VA_IN0">

Commit message: created gerber files for adc and load cell board and did some retouch on load cell board
Routing:
- net VA_IN4: track 9.14 -> 7.82 mm
- net VB_IN4: track 9.11 -> 7.82 mm
- net VDRIVE: track 77.0 -> 76.1 mm
- net N$3: track 9.30 -> 9.88 mm
Changed lines of the file:
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@@
 </class>
 </classes>
-<designrules name="default">
+<designrules name="pban_5mil-l2">
 <description language="de">&lt;b&gt;EAGLE Design Rules&lt;/b&gt;
 &lt;p&gt;
@@
 <param name="layerSetup" value="(1*16)"/>
 <param name="mtCopper" value="0.035mm 0.035mm 0.035mm 0.035mm 0.035mm 0.035mm 0.035mm 0.035mm 0.035mm 0.035mm 0.035mm 0.035mm 0.035mm 0.035mm 0.035mm 0.035mm"/>
-<param name="mtIsolate" value="1.5mm 0.15mm 0.2mm 0.15mm 0.2mm 0.15mm 0.2mm 0.15mm 0.2mm 0.15mm 0.2mm 0.15mm 0.2mm 0.15mm 0.2mm"/>
-<param name="mdWireWire" value="8mil"/>
-<param name="mdWirePad" value="8mil"/>
-<param name="mdWireVia" value="8mil"/>
-<param name="mdPadPad" value="8mil"/>
-<param name="mdPadVia" value="8mil"/>
-<param name="mdViaVia" value="8mil"/>
-<param name="mdSmdPad" value="8mil"/>
-<param name="mdSmdVia" value="8mil"/>
-<param name="mdSmdSmd" value="8mil"/>
-<param name="mdViaViaSameLayer" value="8mil"/>
+<param name="mtIsolate" value="1.53mm 1.5mm 0.2mm 0.15mm 0.2mm 0.15mm 0.2mm 0.15mm 0.2mm 0.15mm 0.2mm 0.15mm 0.2mm 0.15mm 0.2mm"/>
+<param name="mdWireWire" value="5mil"/>
+<param name="mdWirePad" value="0.229mm"/>
+<param name="mdWireVia" value="0.229mm"/>
+<param name="mdPadPad" value="5mil"/>
+<param name="mdPadVia" value="0.229mm"/>
+<param name="mdViaVia" value="5mil"/>
+<param name="mdSmdPad" value="5mil"/>
+<param name="mdSmdVia" value="5mil"/>
+<param name="mdSmdSmd" value="5mil"/>
+<param name="mdViaViaSameLayer" value="5mil"/>
 <param name="mnLayersViaInSmd" value="2"/>
-<param name="mdCopperDimension" value="40mil"/>
-<param name="mdDrill" value="8mil"/>
+<param name="mdCopperDimension" value="0.5mm"/>
+<param name="mdDrill" value="0.5mm"/>
 <param name="mdSmdStop" value="0mil"/>
-<param name="msWidth" value="10mil"/>
-<param name="msDrill" value="24mil"/>
-<param name="msMicroVia" value="9.99mm"/>
-<param name="msBlindViaRatio" value="0.5"/>
+<param name="msWidth" value="5mil"/>
+<param name="msDrill" value="0.3mm"/>
+<param name="msMicroVia" value="0.1mm"/>
+<param name="msBlindViaRatio" value="0.76"/>
 <param name="rvPadTop" value="0.25"/>
 <param name="rvPadInner" value="0.25"/>
@@
 <param name="rvMicroViaOuter" value="0.25"/>
 <param name="rvMicroViaInner" value="0.25"/>
-<param name="rlMinPadTop" value="10mil"/>
-<param name="rlMaxPadTop" value="20mil"/>
-<param name="rlMinPadInner" value="10mil"/>
-<param name="rlMaxPadInner" value="20mil"/>
-<param name="rlMinPadBottom" value="10mil"/>
-<param name="rlMaxPadBottom" value="20mil"/>
-<param name="rlMinViaOuter" value="8mil"/>
-<param name="rlMaxViaOuter" value="20mil"/>
-<param name="rlMinViaInner" value="8mil"/>
-<param name="rlMaxViaInner" value="20mil"/>
-<param name="rlMinMicroViaOuter" value="4mil"/>
-<param name="rlMaxMicroViaOuter" value="20mil"/>
-<param name="rlMinMicroViaInner" value="4mil"/>
-<param name="rlMaxMicroViaInner" value="20mil"/>
+<param name="rlMinPadTop" value="0.15mm"/>
+<param name="rlMaxPadTop" value="0.5mm"/>
+<param name="rlMinPadInner" value="0.2mm"/>
+<param name="rlMaxPadInner" value="0.5mm"/>
+<param name="rlMinPadBottom" value="0.15mm"/>
+<param name="rlMaxPadBottom" value="0.5mm"/>
+<param name="rlMinViaOuter" value="0.15mm"/>
+<param name="rlMaxViaOuter" value="0.5mm"/>
+<param name="rlMinViaInner" value="0.2mm"/>
+<param name="rlMaxViaInner" value="0.5mm"/>
+<param name="rlMinMicroViaOuter" value="0.1mm"/>
+<param name="rlMaxMicroViaOuter" value="0.5mm"/>
+<param name="rlMinMicroViaInner" value="0.1mm"/>
+<param name="rlMaxMicroViaInner" value="0.5mm"/>
 <param name="psTop" value="-1"/>
 <param name="psBottom" value="-1"/>
@@
 <param name="mlMinCreamFrame" value="0mil"/>
 <param name="mlMaxCreamFrame" value="0mil"/>
-<param name="mlViaStopLimit" value="0mil"/>
+<param name="mlViaStopLimit" value="0.35mm"/>
 <param name="srRoundness" value="0"/>
 <param name="srMinRoundness" value="0mil"/>
@@
 <contactref element="U3" pad="52"/>
 <via x="36.3" y="31.45" extent="1-16" drill="0.7"/>
-<via x="30.55" y="12.35" extent="1-16" drill="0.7"/>
-<via x="50.05" y="12.35" extent="1-16" drill="0.7"/>
-<via x="33.15" y="9.1" extent="1-16" drill="0.7"/>
-<via x="47.45" y="9.1" extent="1-16" drill="0.7"/>
 <contactref element="U1" pad="3"/>
 </signal>
@@
 <wire x1="41.276" y1="28.421" x2="41.275" y2="28.42" width="0.4064" layer="1"/>
 <wire x1="43.65" y1="31" x2="48.1" y2="31" width="0.4064" layer="1"/>
-<wire x1="48.1" y1="31" x2="54.036784375" y2="31" width="0.4064" layer="1"/>
-<wire x1="54.036784375" y1="31" x2="54.8" y2="30.236784375" width="0.4064" layer="1"/>
-<wire x1="54.8" y1="30.236784375" x2="54.8" y2="27.15" width="0.4064" layer="1"/>
+<wire x1="48.1" y1="31" x2="52.495115625" y2="31" width="0.4064" layer="1"/>
+<wire x1="52.495115625" y1="31" x2="54.8" y2="28.695115625" width="0.4064" layer="1"/>
+<wire x1="54.8" y1="28.695115625" x2="54.8" y2="27.15" width="0.4064" layer="1"/>
 <wire x1="54.8" y1="27.15" x2="54.8" y2="25.05" width="0.4064" layer="1"/>
 <wire x1="41.275" y1="28.42" x2="41.275" y2="30.181084375" width="0.4064" layer="1"/>
@@
 <wire x1="45.825" y1="12.025" x2="46.8" y2="11.05" width="0.4064" layer="1"/>
 <via x="46.8" y="11.05" extent="1-16" drill="0.7"/>
-<wire x1="46.8" y1="11.05" x2="49.05" y2="11.05" width="0.4064" layer="16"/>
-<wire x1="49.05" y1="11.05" x2="50.05" y2="10.05" width="0.4064" layer="16"/>
-<wire x1="50.05" y1="10.05" x2="50.05" y2="7.15" width="0.4064" layer="16"/>
+<wire x1="46.8" y1="11.05" x2="50.05" y2="7.8" width="0.4064" layer="16"/>
+<wire x1="50.05" y1="7.8" x2="50.05" y2="7.15" width="0.4064" layer="16"/>
 <wire x1="50.05" y1="7.15" x2="50.08" y2="7.12" width="0.4064" layer="16"/>
 </signal>
@@
 <wire x1="34.775" y1="13.18" x2="34.775" y2="12.025" width="0.4064" layer="1"/>
 <wire x1="34.775" y1="12.025" x2="33.8" y2="11.05" width="0.4064" layer="1"/>
-<wire x1="33.8" y1="11.05" x2="31.6" y2="11.05" width="0.4064" layer="16"/>
-<wire x1="31.6" y1="11.05" x2="30.55" y2="10" width="0.4064" layer="16"/>
-<wire x1="30.55" y1="10" x2="30.55" y2="7.15" width="0.4064" layer="16"/>
+<wire x1="33.8" y1="11.05" x2="30.55" y2="7.8" width="0.4064" layer="16"/>
+<wire x1="30.55" y1="7.8" x2="30.55" y2="7.15" width="0.4064" layer="16"/>
 <wire x1="30.55" y1="7.15" x2="30.52" y2="7.12" width="0.4064" layer="16"/>
 </signal>
@@
 <contactref element="U3" pad="68"/>
 <contactref element="U1" pad="4"/>
-<wire x1="25.6652" y1="27.9396" x2="26.1604" y2="27.9396" width="0.4064" layer="1"/>
-<wire x1="26.1604" y1="27.9396" x2="31.675" y2="22.425" width="0.4064" layer="1"/>
-<wire x1="32.68" y1="22.425" x2="31.675" y2="22.425" width="0.4064" layer="1"/>
+<wire x1="32.68" y1="22.425" x2="31.175" y2="22.425" width="0.4064" layer="1"/>
+<wire x1="25.6652" y1="27.9396" x2="26.6604" y2="27.9396" width="0.4064" layer="1"/>
+<wire x1="26.6604" y1="27.9396" x2="30.55" y2="24.05" width="0.4064" layer="1"/>
+<wire x1="30.55" y1="24.05" x2="30.55" y2="23.05" width="0.4064" layer="1"/>
+<wire x1="30.55" y1="23.05" x2="31.175" y2="22.425" width="0.4064" layer="1"/>
 </signal>
 </signals>

Commit message: used consistent naming and units for values
Parts:
- C1, C10, C12, C13, C15, C16, C20, C21, C3, C5, C7: value 0.1u -> 100nF
- C11, C14, C17, C18, C19, C2, C4, C6, C8, C9: value 10u -> 10uF
Changed lines of the file:
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@@
 </autorouter>
 <elements>
-<element name="C1" library="rcl" package="C0603" value="0.1u" x="27.6" y="21.35" rot="R90"/>
+<element name="C1" library="rcl" package="C0603" value="100nF" x="27.6" y="21.35" rot="R90"/>
 <element name="SV3" library="con-lsta" package="FE08-2" value="" x="4.55" y="17.55" rot="R270">
 <attribute name="MPN" value="" x="4.55" y="17.55" size="1.778" layer="27" rot="R270" display="off"/>
@@
 <attribute name="VENDOR" value="Vendor" x="12.35" y="5.05" size="1.778" layer="27" display="off"/>
 </element>
-<element name="C13" library="rcl" package="C0603" value="0.1u" x="6.7" y="4.85" rot="R270"/>
-<element name="C14" library="rcl" package="C1206" value="10u" x="3.9" y="4.3" rot="R270"/>
-<element name="C15" library="rcl" package="C0603" value="0.1u" x="17.55" y="3.6" rot="R270"/>
-<element name="C16" library="rcl" package="C0603" value="0.1u" x="16.7" y="11.45" rot="R180"/>
-<element name="C17" library="rcl" package="C1206" value="10u" x="16.15" y="9" rot="R180"/>
+<element name="C13" library="rcl" package="C0603" value="100nF" x="6.7" y="4.85" rot="R270"/>
+<element name="C14" library="rcl" package="C1206" value="10uF" x="3.9" y="4.3" rot="R270"/>
+<element name="C15" library="rcl" package="C0603" value="100nF" x="17.55" y="3.6" rot="R270"/>
+<element name="C16" library="rcl" package="C0603" value="100nF" x="16.7" y="11.45" rot="R180"/>
+<element name="C17" library="rcl" package="C1206" value="10uF" x="16.15" y="9" rot="R180"/>
 <element name="SV5" library="con-lsta" package="FE20-2" value="" x="28.6" y="41.6" rot="MR180">
 <attribute name="MF" value="" x="28.6" y="41.6" size="1.778" layer="28" rot="MR180" display="off"/>
@@
 <attribute name="OC_FARNELL" value="unknown" x="29.25" y="5.85" size="1.778" layer="27" rot="R180" display="off"/>
 </element>
-<element name="C2" library="rcl" package="C0603" value="10u" x="25.4" y="21.35" rot="R90"/>
-<element name="C3" library="rcl" package="C0603" value="0.1u" x="38.05" y="16.9" rot="MR90"/>
-<element name="C4" library="rcl" package="C0603" value="10u" x="34.75" y="16.9" rot="MR90"/>
-<element name="C5" library="rcl" package="C0603" value="0.1u" x="41.6" y="16.9" rot="MR90"/>
-<element name="C6" library="rcl" package="C0603" value="10u" x="44.95" y="16.9" rot="MR90"/>
-<element name="C7" library="rcl" package="C0603" value="0.1u" x="47.75" y="21.75" rot="MR180"/>
-<element name="C8" library="rcl" package="C0603" value="10u" x="47.75" y="19.15" rot="MR180"/>
-<element name="C9" library="rcl" package="C0603" value="10u" x="50.8" y="21.1" rot="R180"/>
-<element name="C10" library="rcl" package="C0603" value="0.1u" x="48.1" y="31.85" rot="R90"/>
-<element name="C11" library="rcl" package="C0603" value="10u" x="43.65" y="31.85" rot="R90"/>
-<element name="C12" library="rcl" package="C0603" value="0.1u" x="38.35" y="23.15" rot="MR180"/>
-<element name="C18" library="rcl" package="C0603" value="10u" x="38.35" y="20.05" rot="MR180"/>
-<element name="C19" library="rcl" package="C0603" value="10u" x="29.45" y="20.05" rot="MR0"/>
-<element name="C20" library="rcl" package="C0603" value="0.1u" x="29.45" y="23.55" rot="MR0"/>
+<element name="C2" library="rcl" package="C0603" value="10uF" x="25.4" y="21.35" rot="R90"/>
+<element name="C3" library="rcl" package="C0603" value="100nF" x="38.05" y="16.9" rot="MR90"/>
+<element name="C4" library="rcl" package="C0603" value="10uF" x="34.75" y="16.9" rot="MR90"/>
+<element name="C5" library="rcl" package="C0603" value="100nF" x="41.6" y="16.9" rot="MR90"/>
+<element name="C6" library="rcl" package="C0603" value="10uF" x="44.95" y="16.9" rot="MR90"/>
+<element name="C7" library="rcl" package="C0603" value="100nF" x="47.75" y="21.75" rot="MR180"/>
+<element name="C8" library="rcl" package="C0603" value="10uF" x="47.75" y="19.15" rot="MR180"/>
+<element name="C9" library="rcl" package="C0603" value="10uF" x="50.8" y="21.1" rot="R180"/>
+<element name="C10" library="rcl" package="C0603" value="100nF" x="48.1" y="31.85" rot="R90"/>
+<element name="C11" library="rcl" package="C0603" value="10uF" x="43.65" y="31.85" rot="R90"/>
+<element name="C12" library="rcl" package="C0603" value="100nF" x="38.35" y="23.15" rot="MR180"/>
+<element name="C18" library="rcl" package="C0603" value="10uF" x="38.35" y="20.05" rot="MR180"/>
+<element name="C19" library="rcl" package="C0603" value="10uF" x="29.45" y="20.05" rot="MR0"/>
+<element name="C20" library="rcl" package="C0603" value="100nF" x="29.45" y="23.55" rot="MR0"/>
 <element name="R1" library="resistor" package="R0603" value="10k" x="53.95" y="27.15"/>
 <element name="R3" library="resistor" package="R0603" value="10k" x="53.95" y="25.05"/>
-<element name="C21" library="rcl" package="C0603" value="0.1u" x="53.95" y="22.95" rot="R180"/>
+<element name="C21" library="rcl" package="C0603" value="100nF" x="53.95" y="22.95" rot="R180"/>
 <element name="R5" library="resistor" package="R0603" value="10k" x="18.4" y="13.85" rot="R180"/>
 <element name="U1" library="74AHC1G04GW" package="SOT65P210X110-5N" value="74AHC1G04GW/T1" x="24.7" y="28.6">
