File: ADC/RPi_Extension_adc.brd (EAGLE design)
At the start: 63 x 50 mm, 47 parts, among them U1 74AHC1G04GW/T1, U2 ADR423ARZ, U3 AD7616BSTZ

Commit message: updated content before making repository public
Parts:
- added S1: (no value), switch-omron:B3F-10XX
- U2: value ADR423ARZ -> ADR421ARZ
- moved C21 2.16 mm to (54.1, 20.8), turned to 90 degrees
Connections:
- net GND: now also S1.3, S1.4
- net N$7: now also S1.1
Routing:
- net N$7: track 5.46 -> 16.7 mm
- net N$10: track 44.0 -> 46.1 mm
