File: Breakout Jetson/RPi_Extension_breakout_jetson_alt.sch (EAGLE design)
At the start: 8 parts, among them U1 CD74HC4067SM96

Commit message: updated package of 1:16 multiplexer
Parts:
- U1: value CD74HC4067SM96 -> Value
Changed lines of the file:
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@@
 <part name="P+3" library="supply1" deviceset="+5V" device=""/>
 <part name="SV1" library="con-lstb" deviceset="MA06-2" device=""/>
-<part name="U1" library="CD74HC4067" deviceset="CD74HC4067SM96" device="" value=""/>
+<part name="U1" library="CD74HC4067" deviceset="CD74HC4067SM96" device="" value="Value"/>
 </parts>
 <sheets>

Commit message: added inverters to jetson tx1 board
Parts:
- added U10, U11, U12, U13, U14, U15, U16, U17, U2, U3, U4, U5, U6, U7, U8, U9: 74AHC1G04GW/T1, 74AHC1G04GW:74AHC1G04GW/T1
Connections:
- new net GPIO0_NEG: SV5.24, U5.Y
- new net GPIO10_NEG: SV5.33, U11.Y
- new net GPIO11_NEG: SV5.31, U2.Y
- new net GPIO12_NEG: SV5.3, U9.Y
- new net GPIO13_NEG: SV5.5, U17.Y
- new net GPIO14_NEG: SV5.10, U8.Y
- new net GPIO15_NEG: SV5.8, U15.Y
- new net GPIO1_NEG: SV5.26, U4.Y
- new net GPIO2_NEG: SV5.32, U3.Y
- new net GPIO3_NEG: SV5.36, U12.Y
- new net GPIO4_NEG: SV5.7, U16.Y
- new net GPIO5_NEG: SV5.11, U7.Y
- new net GPIO6_NEG: SV5.13, U6.Y
- new net GPIO7_NEG: SV5.15, U14.Y
- new net GPIO8_NEG: SV5.37, U13.Y
- new net GPIO9_NEG: SV5.35, U10.Y
- net DVCC: now also U10.VCC, U11.VCC, U12.VCC, U13.VCC, U14.VCC, U15.VCC, U16.VCC, U17.VCC, U2.VCC, U3.VCC, U4.VCC, U5.VCC, U6.VCC, U7.VCC, U8.VCC, U9.VCC
- net GND: now also U10.GND, U11.GND, U12.GND, U13.GND, U14.GND, U15.GND, U16.GND, U17.GND, U2.GND, U3.GND, U4.GND, U5.GND, U6.GND, U7.GND, U8.GND, U9.GND
- net GPIO0: now also U5.A; no longer SV5.24
- net GPIO1: now also U4.A; no longer SV5.26
- net GPIO10: now also U11.A; no longer SV5.33
- net GPIO11: now also U2.A; no longer SV5.31
- net GPIO12: now also U9.A; no longer SV5.3
- net GPIO13: now also U17.A; no longer SV5.5
- net GPIO14: now also U8.A; no longer SV5.10
- net GPIO15: now also U15.A; no longer SV5.8
- net GPIO2: now also U3.A; no longer SV5.32
- net GPIO3: now also U12.A; no longer SV5.36
- net GPIO4: now also U16.A; no longer SV5.7
- net GPIO5: now also U7.A; no longer SV5.11
- net GPIO6: now also U6.A; no longer SV5.13
- net GPIO7: now also U14.A; no longer SV5.15
- net GPIO8: now also U13.A; no longer SV5.37
- net GPIO9: now also U10.A; no longer SV5.35

Commit message: rearranged pins on jetson board for a nicer layout
Connections:
- removed net ADDR4: SV1.10
- removed net ADDR5: SV1.12
- new net IO_SIGNAL: SV1.9, U1.COMMON_I_O
- net ADDR2: now also SV1.11; no longer SV1.6
- net ADDR3: now also SV1.12; no longer SV1.8
- net GND: now also SV1.8, U1.GND
- net MISO: now also SV1.7; no longer SV1.9
- net MOSI: now also SV1.6; no longer SV1.7
- net SCLK: now also SV1.10; no longer SV1.11
Other:
- moved on the sheet: C19, C20, C21, SV1, SV2, U1, U10, U11, U12, U13, U14, U15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
