File: PSU/RPi_Extension_psu.sch (EAGLE design)
At the start: 40 parts, among them U1 ADP2303ARDZ-5.0, U2 TPS54356-EP_PWP_16, X1 MKDSN1,5/3-5,08

Commit message: updated pcbs
Parts:
- C1, C11, C14, C2, C7: value (none) -> 10uF
- C10, C13, C15, C3, C4: value (none) -> 0.1uF
- C12: value (none) -> 1.0uF
- C16: value (none) -> 1500pF
- C22: value (none) -> 220uF
- C23, C24: value (none) -> 100nF
- L1: value (none) -> 4.7uH
- L2: value (none) -> 22uH
- R1: value (none) -> 100k
- R2: value (none) -> 56k
- R3: value (none) -> 10.2k
- R4: value (none) -> 52.3k
- R5: value (none) -> 10k
- R6: value (none) -> 4.7
Other:
- moved on the sheet: C1, C2, C23, C24, C3, C4

Commit message: reworked PSU layout
Parts:
- removed D2: 1SMA5934BT3G, 1sma59xx_10:1SMA5934BT3G
- C10, C13, C15, C3, C4: value 0.1uF -> 100nF
- C17: value 100UF -> 100uF
- C18: value 330UF -> 330uF
- C25, C5: value 680UF -> 680uF
- C8: value (none) -> 47uF
- C9: value (none) -> 100nF
Connections:
- removed net N$10: C13.2, D2.C, L2.1, R6.1, U2.PH, U2.PH_2
- new net VOUT: C13.2, L2.1, MBRS340T3.C, R6.1, U2.PH, U2.PH_2
- net GND: now also MBRS340T3.A; no longer D2.A
Other:
- moved on the sheet: MBRS340T3, U1

Commit message: used consistent naming and units for values
Other:
- moved on the sheet: C1, C14, C15, C18, C19, C2, C20, C21, C25, C3, C4, C5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

Commit message: cleaned up silklayer of psu board
Parts:
- renumbered MBRS340T3 to D2
Changed lines of the file:
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@@
 <part name="C25" library="Panasonic-EEEFT_EEEH" deviceset="EEE-" device="-CASE-F" technology="FT1C681AP" value="680uF"/>
 <part name="C5" library="Panasonic-EEEFT_EEEH" deviceset="EEE-" device="-CASE-F" technology="FT1C681AP" value="680uF"/>
-<part name="MBRS340T3" library="s3x_10" deviceset="S3*" device="" technology="A"/>
+<part name="D2" library="s3x_10" deviceset="S3*" device="" technology="A"/>
 </parts>
 <sheets>
@@
 <instance part="C25" gate="A" x="264.16" y="40.64" rot="R90"/>
 <instance part="C5" gate="A" x="264.16" y="22.86" rot="R90"/>
-<instance part="MBRS340T3" gate="G$1" x="162.56" y="109.22" rot="R90"/>
+<instance part="D2" gate="G$1" x="162.56" y="109.22" rot="R90"/>
 </instances>
 <busses>
@@
 <pinref part="C16" gate="G$1" pin="2"/>
 <junction x="170.18" y="99.06"/>
-<pinref part="MBRS340T3" gate="G$1" pin="A"/>
+<pinref part="D2" gate="G$1" pin="A"/>
 <wire x1="162.56" y1="106.68" x2="162.56" y2="101.6" width="0.1524" layer="91"/>
 <junction x="162.56" y="101.6"/>
@@
 <wire x1="157.48" y1="111.76" x2="157.48" y2="116.84" width="0.1524" layer="91"/>
 <junction x="157.48" y="116.84"/>
-<pinref part="MBRS340T3" gate="G$1" pin="C"/>
+<pinref part="D2" gate="G$1" pin="C"/>
 <wire x1="162.56" y1="111.76" x2="162.56" y2="116.84" width="0.1524" layer="91"/>
 <junction x="162.56" y="116.84"/>

Commit message: added more documentation
Parts:
- C8: value 47uF -> 22uF
- C9: value 100nF -> 22uF
Changed lines of the file:
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@@
 <part name="GND11" library="supply1" deviceset="GND" device=""/>
 <part name="GND12" library="supply1" deviceset="GND" device=""/>
-<part name="X1" library="con-phoenix-508" deviceset="MKDSN1,5/3-5,08" device=""/>
+<part name="X1" library="con-phoenix-508" deviceset="MKDSN1,5/3-5,08" device="" value=""/>
 <part name="GND1" library="supply1" deviceset="GND" device=""/>
 <part name="C1" library="rcl" deviceset="C-EU" device="C1206" value="10uF"/>
@@
 <part name="GND7" library="supply1" deviceset="GND" device=""/>
 <part name="C7" library="rcl" deviceset="C-EU" device="C0603" value="10uF"/>
-<part name="C8" library="rcl" deviceset="C-EU" device="C0603" value="47uF"/>
-<part name="C9" library="rcl" deviceset="C-EU" device="C0603" value="100nF"/>
+<part name="C8" library="rcl" deviceset="C-EU" device="C0603" value="22uF"/>
+<part name="C9" library="rcl" deviceset="C-EU" device="C0603" value="22uF"/>
 <part name="C10" library="rcl" deviceset="C-EU" device="C0603" value="100nF"/>
 <part name="R1" library="rcl" deviceset="R-EU_" device="R0603" value="100k"/>
