File: Mainboard/Mainboard.brd (EAGLE design)
At the start: 310 x 150 mm, 221 parts, among them J1 JST_PH_B3B-PH-K-S(LF)(SN), J10 JST_PH_B3B-PH-K-S(LF)(SN), J11 JST_PH_B3B-PH-K-S(LF)(SN), J12 JST_PH_B3B-PH-K-S(LF)(SN), J13 JST_PH_B3B-PH-K-S(LF)(SN), J14 JST_PH_B3B-PH-K-S(LF)(SN), J15 JST_PH_B3B-PH-K-S(LF)(SN), J16 JST_PH_B3B-PH-K-S(LF)(SN), J17 JST_PH_B3B-PH-K-S(LF)(SN), J18 JST_PH_B3B-PH-K-S(LF)(SN), J19 JST_PH_B3B-PH-K-S(LF)(SN), J2 JST_PH_B3B-PH-K-S(LF)(SN), J20 JST_PH_B3B-PH-K-S(LF)(SN), J21 JST_PH_B3B-PH-K-S(LF)(SN), J22 JST_PH_B3B-PH-K-S(LF)(SN), J23 JST_PH_B3B-PH-K-S(LF)(SN), J24 JST_PH_B3B-PH-K-S(LF)(SN), J25 JST_PH_B3B-PH-K-S(LF)(SN), J26 JST_PH_B3B-PH-K-S(LF)(SN), J27 JST_PH_B3B-PH-K-S(LF)(SN), J28 JST_PH_B3B-PH-K-S(LF)(SN), J29 JST_PH_B3B-PH-K-S(LF)(SN), J3 JST_PH_B3B-PH-K-S(LF)(SN), J30 JST_PH_B3B-PH-K-S(LF)(SN), J31 JST_PH_B3B-PH-K-S(LF)(SN), J32 JST_PH_B3B-PH-K-S(LF)(SN), J4 JST_PH_B3B-PH-K-S(LF)(SN), J5 JST_PH_B3B-PH-K-S(LF)(SN), J6 JST_PH_B3B-PH-K-S(LF)(SN), J7 JST_PH_B3B-PH-K-S(LF)(SN), J8 JST_PH_B3B-PH-K-S(LF)(SN), J9 JST_PH_B3B-PH-K-S(LF)(SN), U15 AD5360BSTZ, U16 ADR425ARZ, U18 AD7730BRUZ, U19 AD5360BSTZ, U20 ADR425ARZ, U21 AD7730BRUZ, U22 STM32F103RCT6, U23 AD7730BRUZ, U24 AD7730BRUZ, U25 AD7730BRUZ, U26 AD7730BRUZ, U27 AD7730BRUZ, U28 AD7730BRUZ, U38 AD7730BRUZ, U39 AD7730BRUZ, U4 ADR421ARZ, U40 STM32F103RCT6, U41 AD7730BRUZ, U42 AD7730BRUZ, U43 AD7730BRUZ, U44 AD7730BRUZ, U45 AD7730BRUZ, U46 AD7730BRUZ, U5 AD7616BSTZ, U6 74AHC1G04GW/T1, U7 ADR421ARZ, U8 AD7616BSTZ, U9 74AHC1G04GW/T1, Y3 KC2520B-C1, Y4 ABM3B, Y7 KC2520B-C1, Y8 ABM3B

Commit message: added RPi power supply
Parts:
- added JP1: (no value), jumper:JP1
- R1, R5: value (none) -> 220
- R10: value (none) -> 680
- R3: value (none) -> 68
- moved S1 7.18 mm to (282.8, 131.3)
Connections:
- new net N$1: JP1.2, SV1.2, SV1.4
- net +5V: now also JP1.1
Routing:
- net +5V: track 1103.7 -> 1444.8 mm
- net SCLK: track 693.5 -> 681.9 mm, vias 6 -> 4
- net N$1: track 0.00 -> 7.27 mm
- net SS_ADC_1: track 129.8 -> 135.2 mm
- net CONVST: track 166.3 -> 161.2 mm
- net MOSI: track 712.5 -> 709.0 mm
- net MISO: track 703.0 -> 699.8 mm
- net DVCC: track 1355.6 -> 1358.7 mm
- net PSU_ENABLE: track 98.0 -> 100.3 mm
Other:
- board text added: "+12V"
- board text added: "+3.3V"
- board text added: "+5V"
- board text added: "OFF"
- board text added: "ON"
- board text added: "PWR_GOOD"

Commit message: added fan and leds
Parts:
- added LED5: (no value), led:LED3MM
- added R11: 330, resistor:R0805
- added X1: 22-23-2031, con-molex:22-23-2031
Connections:
- new net HEARTBEAT: R11.2, SV1.3
- new net N$6: LED5.A, R11.1
- net GND: now also LED5.K, X1.3
- net VDD: now also X1.2
Routing:
- net VDD: track 954.5 -> 992.7 mm
- net HEARTBEAT: track 0.00 -> 14.6 mm
- net N$6: track 0.00 -> 4.70 mm
- net SS_ADC_2: track 30.9 -> 33.8 mm
- net DVCC: track 1358.7 -> 1360.6 mm
Other:
- board text added: "1"
- board text added: "16"
- board text added: "17"
- board text added: "32"
- board text added: "Fan"
- board text added: "Heartbeat"
- board text added: "RPi3"

Commit message: now using polarized symbol for tantalum caps
Parts:
- removed C104, C105, C106, C108, C110, C112, C115, C118, C138, C139, C140, C142, C144, C146, C149, C152, C34, C37, C65, C68: 10uF, rcl:C1206
- added C1, C10, C2, C21, C22, C23, C24, C25, C26, C27, C28, C29, C3, C30, C4, C5, C6, C7, C8, C9: 10uF, resistor:SMC_A
Connections:
- net ADC_1_VREF: now also C28.+; no longer C37.1
- net ADC_2_VREF: now also C30.+; no longer C68.1
- net DVCC: now also C1.+, C2.+, C21.+, C22.+; no longer C104.1, C105.1, C138.1, C139.1
- net GND: now also C1.-, C10.-, C2.-, C21.-, C22.-, C23.-, C24.-, C25.+, C26.+, C27.-, C28.-, C29.-, C3.-, C30.-, C4.-, C5.-, C6.-, C7.+, C8.+, C9.-; no longer C104.2, C105.2, C106.2, C108.2, C110.2, C112.2, C115.2, C118.2, C138.2, C139.2, C140.2, C142.2, C144.2, C146.2, C149.2, C152.2, C34.2, C37.2, C65.2, C68.2
- net VDD: now also C23.+, C24.+, C27.+, C29.+, C3.+, C5.+, C6.+, C9.+; no longer C106.1, C108.1, C115.1, C140.1, C142.1, C149.1, C34.1, C65.1
- net VREF_1: now also C4.+; no longer C118.1
- net VREF_2: now also C10.+; no longer C152.1
- net VSS: now also C25.-, C26.-, C7.-, C8.-; no longer C110.1, C112.1, C144.1, C146.1
Routing:
- net VDD: track 992.7 -> 977.9 mm
Other:
- board text added: "Hitzmann 2018 rev. 1.0"
- board text added: "Robot Controller Board"
