File: Mainboard/Mainboard.brd (EAGLE design)
At the start: 310 x 150 mm, 225 parts, among them J1 JST_PH_B3B-PH-K-S(LF)(SN), J10 JST_PH_B3B-PH-K-S(LF)(SN), J11 JST_PH_B3B-PH-K-S(LF)(SN), J12 JST_PH_B3B-PH-K-S(LF)(SN), J13 JST_PH_B3B-PH-K-S(LF)(SN), J14 JST_PH_B3B-PH-K-S(LF)(SN), J15 JST_PH_B3B-PH-K-S(LF)(SN), J16 JST_PH_B3B-PH-K-S(LF)(SN), J17 JST_PH_B3B-PH-K-S(LF)(SN), J18 JST_PH_B3B-PH-K-S(LF)(SN), J19 JST_PH_B3B-PH-K-S(LF)(SN), J2 JST_PH_B3B-PH-K-S(LF)(SN), J20 JST_PH_B3B-PH-K-S(LF)(SN), J21 JST_PH_B3B-PH-K-S(LF)(SN), J22 JST_PH_B3B-PH-K-S(LF)(SN), J23 JST_PH_B3B-PH-K-S(LF)(SN), J24 JST_PH_B3B-PH-K-S(LF)(SN), J25 JST_PH_B3B-PH-K-S(LF)(SN), J26 JST_PH_B3B-PH-K-S(LF)(SN), J27 JST_PH_B3B-PH-K-S(LF)(SN), J28 JST_PH_B3B-PH-K-S(LF)(SN), J29 JST_PH_B3B-PH-K-S(LF)(SN), J3 JST_PH_B3B-PH-K-S(LF)(SN), J30 JST_PH_B3B-PH-K-S(LF)(SN), J31 JST_PH_B3B-PH-K-S(LF)(SN), J32 JST_PH_B3B-PH-K-S(LF)(SN), J4 JST_PH_B3B-PH-K-S(LF)(SN), J5 JST_PH_B3B-PH-K-S(LF)(SN), J6 JST_PH_B3B-PH-K-S(LF)(SN), J7 JST_PH_B3B-PH-K-S(LF)(SN), J8 JST_PH_B3B-PH-K-S(LF)(SN), J9 JST_PH_B3B-PH-K-S(LF)(SN), U15 AD5360BSTZ, U16 ADR425ARZ, U18 AD7730BRUZ, U19 AD5360BSTZ, U20 ADR425ARZ, U21 AD7730BRUZ, U22 STM32F103RCT6, U23 AD7730BRUZ, U24 AD7730BRUZ, U25 AD7730BRUZ, U26 AD7730BRUZ, U27 AD7730BRUZ, U28 AD7730BRUZ, U38 AD7730BRUZ, U39 AD7730BRUZ, U4 ADR421ARZ, U40 STM32F103RCT6, U41 AD7730BRUZ, U42 AD7730BRUZ, U43 AD7730BRUZ, U44 AD7730BRUZ, U45 AD7730BRUZ, U46 AD7730BRUZ, U5 AD7616BSTZ, U6 74AHC1G04GW/T1, U7 ADR421ARZ, U8 AD7616BSTZ, U9 74AHC1G04GW/T1, X1 22-23-2031, Y3 KC2520B-C1, Y4 ABM3B, Y7 KC2520B-C1, Y8 ABM3B

Commit message: minor changes
Parts:
- S1: value 1MS1T1B1M2QES-5 -> (none)
- moved JP1 0.65 mm to (12.2, 147.1)
Routing:
- net N$1: track 7.27 -> 7.90 mm
Other:
- board text added: "Hitzmann 2018 rev. 1.1"
- board text removed: "Hitzmann 2018 rev. 1.0"
Changed lines of the file:
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@@
 <?xml version="1.0" encoding="utf-8"?>
 <!DOCTYPE eagle SYSTEM "eagle.dtd">
-<eagle version="8.7.0">
+<eagle version="8.7.1">
 <drawing>
 <settings>
@@
 <hole x="89.05" y="45.8" drill="5"/>
 <text x="17.55" y="20.15" size="1.778" layer="26" rot="MR0">Robot Controller Board</text>
-<text x="17.55" y="16.25" size="1.778" layer="26" rot="MR0">Hitzmann 2018 rev. 1.0</text>
+<text x="17.55" y="16.25" size="1.778" layer="26" rot="MR0">Hitzmann 2018 rev. 1.1</text>
 </plain>
 <attributes>
@@
 <attribute name="SUPPLIER_NAME" value="RS" x="269.1" y="81.9" size="1.778" layer="27" rot="R90" display="off"/>
 </element>
-<element name="S1" library="1MS1T1B1M2QES-5" package="1MS1T1B1M2QES-5" value="1MS1T1B1M2QES-5" x="282.75" y="131.3" smashed="yes" rot="R270">
+<element name="S1" library="1MS1T1B1M2QES-5" package="1MS1T1B1M2QES-5" value="" x="282.75" y="131.3" smashed="yes" rot="R270">
 <attribute name="3D_PACKAGE" value="" x="282.75" y="131.3" size="1.778" layer="27" rot="R270" display="off"/>
 <attribute name="ALLIED_NUMBER" value="" x="282.75" y="131.3" size="1.778" layer="27" rot="R270" display="off"/>
@@
 <attribute name="VALUE" x="289.31" y="105.285" size="1.27" layer="27" rot="R270"/>
 </element>
-<element name="JP1" library="jumper" library_urn="urn:adsk.eagle:library:252" package="JP1" package3d_urn="urn:adsk.eagle:package:15455/1" value="" x="12.25" y="147.7" rot="R90"/>
+<element name="JP1" library="jumper" library_urn="urn:adsk.eagle:library:252" package="JP1" package3d_urn="urn:adsk.eagle:package:15455/1" value="" x="12.25" y="147.05" rot="R90"/>
 <element name="X1" library="con-molex" library_urn="urn:adsk.eagle:library:165" package="22-23-2031" value="22-23-2031" x="-2.6" y="50.7" rot="R270">
 <attribute name="MF" value="MOLEX" x="-2.6" y="50.7" size="1.778" layer="27" rot="R270" display="off"/>
@@
 <contactref element="C29" pad="-"/>
 <contactref element="C30" pad="-"/>
+<via x="161.85" y="146.9" extent="1-16" drill="0.7"/>
+<via x="161.85" y="144.3" extent="1-16" drill="0.7"/>
+<via x="173.55" y="144.3" extent="1-16" drill="0.7"/>
+<via x="173.55" y="146.9" extent="1-16" drill="0.7"/>
 </signal>
 <signal name="MISO">
@@
 <wire x1="274.3" y1="75.4" x2="273.65" y2="75.4" width="0.4064" layer="1"/>
 <contactref element="JP1" pad="1"/>
-<wire x1="13.52" y1="147.7" x2="154.55" y2="147.7" width="1.27" layer="1"/>
-<wire x1="154.55" y1="147.7" x2="160.55" y2="141.7" width="1.27" layer="1"/>
+<wire x1="13.52" y1="147.05" x2="155.2" y2="147.05" width="1.27" layer="1"/>
+<wire x1="161.2" y1="141.05" x2="155.2" y2="147.05" width="1.27" layer="1"/>
 <wire x1="294.45" y1="85.15" x2="297.7" y2="88.4" width="1.27" layer="1"/>
 <wire x1="297.7" y1="88.4" x2="297.7" y2="135.85" width="1.27" layer="1"/>
-<wire x1="297.7" y1="135.85" x2="291.85" y2="141.7" width="1.27" layer="1"/>
-<wire x1="291.85" y1="141.7" x2="160.55" y2="141.7" width="1.27" layer="1"/>
+<wire x1="297.7" y1="135.85" x2="292.5" y2="141.05" width="1.27" layer="1"/>
 <wire x1="223.925" y1="103.025" x2="220.7806" y2="103.025" width="0.254" layer="16"/>
 <wire x1="226.4194" y1="104.325003125" x2="225.225003125" y2="104.325003125" width="0.254" layer="16"/>
@@
 <wire x1="226.4194" y1="26.325003125" x2="225.225003125" y2="26.325003125" width="0.254" layer="16"/>
 <wire x1="225.225003125" y1="26.325003125" x2="223.925" y2="25.025" width="0.254" layer="16"/>
+<wire x1="292.5" y1="141.05" x2="161.2" y2="141.05" width="1.27" layer="1"/>
 </signal>
 <signal name="DVCC">
@@
 <contactref element="U22" pad="46"/>
 <wire x1="246.485" y1="126.8932" x2="248.2568" y2="126.8932" width="0.254" layer="16"/>
-<wire x1="248.2568" y1="126.8932" x2="248.3" y2="126.9" width="0.254" layer="16"/>
-<via x="248.3" y="126.9" extent="1-16" drill="0.7"/>
+<wire x1="248.2568" y1="126.8932" x2="248.3" y2="127" width="0.254" layer="16"/>
+<via x="248.3" y="127" extent="1-16" drill="0.7"/>
 <contactref element="SV10" pad="6"/>
 <wire x1="258.73" y1="138.39" x2="251.724921875" y2="138.39" width="0.254" layer="1"/>
 <wire x1="251.724921875" y1="138.39" x2="248.3" y2="134.965078125" width="0.254" layer="1"/>
-<wire x1="248.3" y1="134.965078125" x2="248.3" y2="126.9" width="0.254" layer="1"/>
+<wire x1="248.3" y1="134.965078125" x2="248.3" y2="127" width="0.254" layer="1"/>
 </signal>
 <signal name="LC_1_SWDCLK">
@@
 <wire x1="240.7" y1="116.8" x2="241.15" y2="116.35" width="0.254" layer="16"/>
 <contactref element="U22" pad="42"/>
-<via x="248.3" y="124.4" extent="1-16" drill="0.7"/>
+<via x="248.3" y="124.3" extent="1-16" drill="0.7"/>
 <wire x1="245.7" y1="123.5" x2="245.7" y2="120.9" width="0.254" layer="1"/>
 <wire x1="242.75" y1="115.4" x2="242.75" y2="117.95" width="0.254" layer="1"/>
 <wire x1="242.75" y1="117.95" x2="245.7" y2="120.9" width="0.254" layer="1"/>
-<wire x1="248.3" y1="124.4" x2="247.788" y2="124.912" width="0.254" layer="16"/>
-<wire x1="247.788" y1="124.912" x2="246.485" y2="124.912" width="0.254" layer="16"/>
-<wire x1="248.3" y1="124.4" x2="246.6" y2="124.4" width="0.254" layer="1"/>
-<wire x1="246.6" y1="124.4" x2="245.7" y2="123.5" width="0.254" layer="1"/>
+<wire x1="246.485" y1="124.912" x2="247.688" y2="124.912" width="0.254" layer="16"/>
+<wire x1="247.688" y1="124.912" x2="248.3" y2="124.3" width="0.254" layer="16"/>
+<wire x1="248.3" y1="124.3" x2="246.5" y2="124.3" width="0.254" layer="1"/>
+<wire x1="246.5" y1="124.3" x2="245.7" y2="123.5" width="0.254" layer="1"/>
 </signal>
 <signal name="LC_1_RDY6">
@@
 <via x="255.9" y="106.9" extent="1-16" drill="0.7"/>
 <contactref element="U22" pad="17"/>
-<via x="260.5" y="100.5" extent="1-16" drill="0.7"/>
+<via x="260.15" y="100.5" extent="1-16" drill="0.7"/>
 <wire x1="255.9" y1="106.9" x2="255.9" y2="103.35" width="0.254" layer="1"/>
 <wire x1="262.086728125" y1="115.139059375" x2="262.086728125" y2="100.886728125" width="0.254" layer="16"/>
 <wire x1="262.086728125" y1="100.886728125" x2="261.7" y2="100.5" width="0.254" layer="16"/>
-<wire x1="261.7" y1="100.5" x2="260.5" y2="100.5" width="0.254" layer="16"/>
+<wire x1="261.7" y1="100.5" x2="260.15" y2="100.5" width="0.254" layer="16"/>
 <wire x1="255.9592" y1="118.435" x2="258.7907875" y2="118.435" width="0.254" layer="16"/>
 <wire x1="258.7907875" y1="118.435" x2="262.086728125" y2="115.139059375" width="0.254" layer="16"/>
-<wire x1="260.5" y1="100.5" x2="258.75" y2="100.5" width="0.254" layer="1"/>
+<wire x1="260.15" y1="100.5" x2="258.75" y2="100.5" width="0.254" layer="1"/>
 <wire x1="258.75" y1="100.5" x2="255.9" y2="103.35" width="0.254" layer="1"/>
 </signal>
@@
 <contactref element="U40" pad="46"/>
 <wire x1="246.485" y1="48.8932" x2="248.2568" y2="48.8932" width="0.254" layer="16"/>
-<wire x1="248.2568" y1="48.8932" x2="248.3" y2="48.9" width="0.254" layer="16"/>
-<via x="248.3" y="48.9" extent="1-16" drill="0.7"/>
+<wire x1="248.2568" y1="48.8932" x2="248.3" y2="49" width="0.254" layer="16"/>
+<via x="248.3" y="49" extent="1-16" drill="0.7"/>
 <contactref element="SV21" pad="6"/>
 <wire x1="258.73" y1="60.39" x2="251.724921875" y2="60.39" width="0.254" layer="1"/>
 <wire x1="251.724921875" y1="60.39" x2="248.3" y2="56.965078125" width="0.254" layer="1"/>
-<wire x1="248.3" y1="56.965078125" x2="248.3" y2="48.9" width="0.254" layer="1"/>
+<wire x1="248.3" y1="56.965078125" x2="248.3" y2="49" width="0.254" layer="1"/>
 </signal>
 <signal name="LC_2_SWDCLK">
@@
 <wire x1="240.7" y1="38.8" x2="241.15" y2="38.35" width="0.254" layer="16"/>
 <contactref element="U40" pad="42"/>
-<via x="248.3" y="46.4" extent="1-16" drill="0.7"/>
+<via x="248.3" y="46.3" extent="1-16" drill="0.7"/>
 <wire x1="245.7" y1="45.5" x2="245.7" y2="42.9" width="0.254" layer="1"/>
 <wire x1="242.75" y1="37.4" x2="242.75" y2="39.95" width="0.254" layer="1"/>
 <wire x1="242.75" y1="39.95" x2="245.7" y2="42.9" width="0.254" layer="1"/>
-<wire x1="248.3" y1="46.4" x2="247.788" y2="46.912" width="0.254" layer="16"/>
-<wire x1="247.788" y1="46.912" x2="246.485" y2="46.912" width="0.254" layer="16"/>
-<wire x1="248.3" y1="46.4" x2="246.6" y2="46.4" width="0.254" layer="1"/>
-<wire x1="246.6" y1="46.4" x2="245.7" y2="45.5" width="0.254" layer="1"/>
+<wire x1="248.3" y1="46.3" x2="246.5" y2="46.3" width="0.254" layer="1"/>
+<wire x1="246.5" y1="46.3" x2="245.7" y2="45.5" width="0.254" layer="1"/>
+<wire x1="246.485" y1="46.912" x2="247.688" y2="46.912" width="0.254" layer="16"/>
+<wire x1="247.688" y1="46.912" x2="248.3" y2="46.3" width="0.254" layer="16"/>
 </signal>
 <signal name="LC_2_RDY6">
@@
 <via x="255.9" y="28.9" extent="1-16" drill="0.7"/>
 <contactref element="U40" pad="17"/>
-<via x="260.5" y="22.5" extent="1-16" drill="0.7"/>
+<via x="260.15" y="22.5" extent="1-16" drill="0.7"/>
 <wire x1="255.9" y1="28.9" x2="255.9" y2="26.65" width="0.254" layer="1"/>
-<wire x1="260.5" y1="22.5" x2="260.4" y2="22.5" width="0.254" layer="16"/>
+<wire x1="260.15" y1="22.5" x2="260.4" y2="22.5" width="0.254" layer="16"/>
 <wire x1="261.7" y1="22.5" x2="262.35" y2="23.15" width="0.254" layer="16"/>
 <wire x1="262.35" y1="23.15" x2="262.35" y2="36.8757875" width="0.254" layer="16"/>
@@
 <wire x1="255.9" y1="26" x2="255.9" y2="26.65" width="0.254" layer="1"/>
 <wire x1="255.9" y1="25.55" x2="255.9" y2="26" width="0.254" layer="1"/>
-<wire x1="260.5" y1="22.5" x2="258.95" y2="22.5" width="0.254" layer="1"/>
+<wire x1="260.15" y1="22.5" x2="258.95" y2="22.5" width="0.254" layer="1"/>
 <wire x1="258.95" y1="22.5" x2="255.9" y2="25.55" width="0.254" layer="1"/>
-<wire x1="260.5" y1="22.5" x2="261.7" y2="22.5" width="0.254" layer="16"/>
+<wire x1="260.15" y1="22.5" x2="261.7" y2="22.5" width="0.254" layer="16"/>
 </signal>
 <signal name="LC_2_RDY4">
@@
 <wire x1="13.51" y1="142.97" x2="10.97" y2="142.97" width="1.27" layer="1"/>
 <wire x1="10.97" y1="142.97" x2="10.97" y2="147.69" width="1.27" layer="1"/>
-<wire x1="10.97" y1="147.69" x2="10.98" y2="147.7" width="1.27" layer="1"/>
+<wire x1="10.97" y1="147.69" x2="10.98" y2="147.05" width="1.27" layer="1"/>
 </signal>
 <signal name="N$6">
