File: Mainboard/Mainboard.sch (EAGLE design)
At the start: 221 parts, among them J1 JST_PH_B3B-PH-K-S(LF)(SN), J10 JST_PH_B3B-PH-K-S(LF)(SN), J11 JST_PH_B3B-PH-K-S(LF)(SN), J12 JST_PH_B3B-PH-K-S(LF)(SN), J13 JST_PH_B3B-PH-K-S(LF)(SN), J14 JST_PH_B3B-PH-K-S(LF)(SN), J15 JST_PH_B3B-PH-K-S(LF)(SN), J16 JST_PH_B3B-PH-K-S(LF)(SN), J17 JST_PH_B3B-PH-K-S(LF)(SN), J18 JST_PH_B3B-PH-K-S(LF)(SN), J19 JST_PH_B3B-PH-K-S(LF)(SN), J2 JST_PH_B3B-PH-K-S(LF)(SN), J20 JST_PH_B3B-PH-K-S(LF)(SN), J21 JST_PH_B3B-PH-K-S(LF)(SN), J22 JST_PH_B3B-PH-K-S(LF)(SN), J23 JST_PH_B3B-PH-K-S(LF)(SN), J24 JST_PH_B3B-PH-K-S(LF)(SN), J25 JST_PH_B3B-PH-K-S(LF)(SN), J26 JST_PH_B3B-PH-K-S(LF)(SN), J27 JST_PH_B3B-PH-K-S(LF)(SN), J28 JST_PH_B3B-PH-K-S(LF)(SN), J29 JST_PH_B3B-PH-K-S(LF)(SN), J3 JST_PH_B3B-PH-K-S(LF)(SN), J30 JST_PH_B3B-PH-K-S(LF)(SN), J31 JST_PH_B3B-PH-K-S(LF)(SN), J32 JST_PH_B3B-PH-K-S(LF)(SN), J33 B4B-PH-K-S(LF)(SN), J34 B4B-PH-K-S(LF)(SN), J35 B4B-PH-K-S(LF)(SN), J36 B4B-PH-K-S(LF)(SN), J37 B4B-PH-K-S(LF)(SN), J38 B4B-PH-K-S(LF)(SN), J39 B4B-PH-K-S(LF)(SN), J4 JST_PH_B3B-PH-K-S(LF)(SN), J40 B4B-PH-K-S(LF)(SN), J41 B4B-PH-K-S(LF)(SN), J42 B4B-PH-K-S(LF)(SN), J43 B4B-PH-K-S(LF)(SN), J44 B4B-PH-K-S(LF)(SN), J45 B4B-PH-K-S(LF)(SN), J46 B4B-PH-K-S(LF)(SN), J47 B4B-PH-K-S(LF)(SN), J48 B4B-PH-K-S(LF)(SN), J49 B4B-PH-K-S(LF)(SN), J5 JST_PH_B3B-PH-K-S(LF)(SN), J50 B4B-PH-K-S(LF)(SN), J51 B4B-PH-K-S(LF)(SN), J52 B4B-PH-K-S(LF)(SN), J53 B4B-PH-K-S(LF)(SN), J54 B4B-PH-K-S(LF)(SN), J55 B4B-PH-K-S(LF)(SN), J56 B4B-PH-K-S(LF)(SN), J57 B4B-PH-K-S(LF)(SN), J58 B4B-PH-K-S(LF)(SN), J59 B4B-PH-K-S(LF)(SN), J6 JST_PH_B3B-PH-K-S(LF)(SN), J60 B4B-PH-K-S(LF)(SN), J61 B4B-PH-K-S(LF)(SN), J62 B4B-PH-K-S(LF)(SN), J63 B4B-PH-K-S(LF)(SN), J64 B4B-PH-K-S(LF)(SN), J7 JST_PH_B3B-PH-K-S(LF)(SN), J8 JST_PH_B3B-PH-K-S(LF)(SN), J9 JST_PH_B3B-PH-K-S(LF)(SN), U1 AMP-5103309-7-34PIN_5103309-7, U15 AD5360BSTZ, U16 ADR425ARZ, U18 AD7730BRUZ, U19 AD5360BSTZ, U2 AMP-5103309-7-34PIN_5103309-7, U20 ADR425ARZ, U21 AD7730BRUZ, U22 STM32F103RCT6, U23 AD7730BRUZ, U24 AD7730BRUZ, U25 AD7730BRUZ, U26 AD7730BRUZ, U27 AD7730BRUZ, U28 AD7730BRUZ, U38 AD7730BRUZ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

Commit message: added RPi power supply
Parts:
- added JP1: (no value), jumper:JP1Q
- R1, R5: value (none) -> 220
- R10: value (none) -> 680
- R3: value (none) -> 68
Connections:
- new net N$1: JP1.2, SV1.2, SV1.4
- net +5V: now also JP1.1
Changed lines of the file:
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@@
 <part name="LED4" library="led" library_urn="urn:adsk.eagle:library:259" deviceset="TLLG4400" device="" package3d_urn="urn:adsk.eagle:package:15797/1" value=""/>
 <part name="GND136" library="supply1" library_urn="urn:adsk.eagle:library:371" deviceset="GND" device=""/>
-<part name="R1" library="resistor" library_urn="urn:adsk.eagle:library:348" deviceset="R-EU_" device="R0805" package3d_urn="urn:adsk.eagle:package:26059/1"/>
-<part name="R3" library="resistor" library_urn="urn:adsk.eagle:library:348" deviceset="R-EU_" device="R0805" package3d_urn="urn:adsk.eagle:package:26059/1"/>
-<part name="R5" library="resistor" library_urn="urn:adsk.eagle:library:348" deviceset="R-EU_" device="R0805" package3d_urn="urn:adsk.eagle:package:26059/1"/>
-<part name="R10" library="resistor" library_urn="urn:adsk.eagle:library:348" deviceset="R-EU_" device="R0805" package3d_urn="urn:adsk.eagle:package:26059/1"/>
+<part name="R1" library="resistor" library_urn="urn:adsk.eagle:library:348" deviceset="R-EU_" device="R0805" package3d_urn="urn:adsk.eagle:package:26059/1" value="220"/>
+<part name="R3" library="resistor" library_urn="urn:adsk.eagle:library:348" deviceset="R-EU_" device="R0805" package3d_urn="urn:adsk.eagle:package:26059/1" value="68"/>
+<part name="R5" library="resistor" library_urn="urn:adsk.eagle:library:348" deviceset="R-EU_" device="R0805" package3d_urn="urn:adsk.eagle:package:26059/1" value="220"/>
+<part name="R10" library="resistor" library_urn="urn:adsk.eagle:library:348" deviceset="R-EU_" device="R0805" package3d_urn="urn:adsk.eagle:package:26059/1" value="680"/>
 <part name="P+54" library="supply1" library_urn="urn:adsk.eagle:library:371" deviceset="+5V" device=""/>
+<part name="JP1" library="jumper" library_urn="urn:adsk.eagle:library:252" deviceset="JP1Q" device="" package3d_urn="urn:adsk.eagle:package:15455/1"/>
+<part name="P+55" library="supply1" library_urn="urn:adsk.eagle:library:371" deviceset="+5V" device=""/>
 </parts>
 <sheets>
@@
 <instance part="GND149" gate="1" x="-25.4" y="238.76"/>
 <instance part="S1" gate="G$1" x="403.86" y="259.08"/>
-<instance part="GND135" gate="1" x="439.42" y="254"/>
+<instance part="GND135" gate="1" x="431.8" y="254"/>
 <instance part="LED3" gate="G$1" x="312.42" y="251.46"/>
 <instance part="LED2" gate="G$1" x="325.12" y="251.46"/>
@@
 <instance part="R10" gate="G$1" x="345.44" y="264.16" rot="R90"/>
 <instance part="P+54" gate="1" x="335.28" y="284.48"/>
+<instance part="JP1" gate="A" x="30.48" y="220.98"/>
+<instance part="P+55" gate="1" x="30.48" y="205.74" rot="R180"/>
 </instances>
 <busses>
@@
 <pinref part="P+54" gate="1" pin="+5V"/>
 </segment>
+<segment>
+<pinref part="P+55" gate="1" pin="+5V"/>
+<pinref part="JP1" gate="A" pin="1"/>
+<wire x1="30.48" y1="208.28" x2="30.48" y2="213.36" width="0.1524" layer="91"/>
+</segment>
 </net>
 <net name="VSS" class="0">
@@
 <segment>
 <pinref part="S1" gate="G$1" pin="3"/>
-<wire x1="424.18" y1="259.08" x2="439.42" y2="259.08" width="0.1524" layer="91"/>
+<wire x1="424.18" y1="259.08" x2="431.8" y2="259.08" width="0.1524" layer="91"/>
 <pinref part="GND135" gate="1" pin="GND"/>
-<wire x1="439.42" y1="259.08" x2="439.42" y2="256.54" width="0.1524" layer="91"/>
+<wire x1="431.8" y1="259.08" x2="431.8" y2="256.54" width="0.1524" layer="91"/>
 </segment>
 <segment>
@@
 </segment>
 </net>
+<net name="N$1" class="0">
+<segment>
+<pinref part="SV1" gate="G$1" pin="4"/>
+<wire x1="20.32" y1="236.22" x2="30.48" y2="236.22" width="0.1524" layer="91"/>
+<wire x1="30.48" y1="236.22" x2="30.48" y2="233.68" width="0.1524" layer="91"/>
+<pinref part="SV1" gate="G$1" pin="2"/>
+<wire x1="30.48" y1="233.68" x2="30.48" y2="228.6" width="0.1524" layer="91"/>
+<wire x1="20.32" y1="233.68" x2="30.48" y2="233.68" width="0.1524" layer="91"/>
+<junction x="30.48" y="233.68"/>
+<pinref part="JP1" gate="A" pin="2"/>
+</segment>
+</net>

Commit message: added fan and leds
Parts:
- added LED5: TLLG4400, led:TLLG4400
- added R11: 330, resistor:R-EU_R0805
- added X1: 22-23-2031, con-molex:22-23-2031
Connections:
- new net HEARTBEAT: R11.2, SV1.3
- new net N$6: LED5.A, R11.1
- net GND: now also LED5.C, X1-3.S
- net VDD: now also X1-2.S
Changed lines of the file:
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@@
 <part name="JP1" library="jumper" library_urn="urn:adsk.eagle:library:252" deviceset="JP1Q" device="" package3d_urn="urn:adsk.eagle:package:15455/1"/>
 <part name="P+55" library="supply1" library_urn="urn:adsk.eagle:library:371" deviceset="+5V" device=""/>
+<part name="X1" library="con-molex" library_urn="urn:adsk.eagle:library:165" deviceset="22-23-2031" device=""/>
+<part name="GND150" library="supply1" library_urn="urn:adsk.eagle:library:371" deviceset="GND" device=""/>
+<part name="LED5" library="led" library_urn="urn:adsk.eagle:library:259" deviceset="TLLG4400" device="" package3d_urn="urn:adsk.eagle:package:15797/1" value=""/>
+<part name="R11" library="resistor" library_urn="urn:adsk.eagle:library:348" deviceset="R-EU_" device="R0805" package3d_urn="urn:adsk.eagle:package:26059/1" value="330"/>
 </parts>
 <sheets>
@@
 <instance part="LED1" gate="G$1" x="335.28" y="251.46"/>
 <instance part="LED4" gate="G$1" x="345.44" y="251.46"/>
-<instance part="GND136" gate="1" x="353.06" y="238.76"/>
+<instance part="GND136" gate="1" x="355.6" y="238.76"/>
 <instance part="R1" gate="G$1" x="312.42" y="264.16" rot="R90"/>
 <instance part="R3" gate="G$1" x="325.12" y="264.16" rot="R90"/>
@@
 <instance part="JP1" gate="A" x="30.48" y="220.98"/>
 <instance part="P+55" gate="1" x="30.48" y="205.74" rot="R180"/>
+<instance part="X1" gate="-1" x="116.84" y="264.16"/>
+<instance part="X1" gate="-2" x="116.84" y="261.62"/>
+<instance part="X1" gate="-3" x="116.84" y="259.08"/>
+<instance part="GND150" gate="1" x="104.14" y="254"/>
+<instance part="LED5" gate="G$1" x="355.6" y="251.46"/>
+<instance part="R11" gate="G$1" x="355.6" y="264.16" rot="R90"/>
 </instances>
 <busses>
@@
 <label x="345.44" y="279.4" size="1.778" layer="95" rot="R90"/>
 </segment>
+<segment>
+<pinref part="X1" gate="-2" pin="S"/>
+<wire x1="114.3" y1="261.62" x2="104.14" y2="261.62" width="0.1524" layer="91"/>
+<label x="99.06" y="261.62" size="1.778" layer="95"/>
+</segment>
 </net>
 <net name="GND" class="0">
@@
 <wire x1="335.28" y1="246.38" x2="345.44" y2="246.38" width="0.1524" layer="91"/>
 <junction x="335.28" y="246.38"/>
-<wire x1="345.44" y1="246.38" x2="353.06" y2="246.38" width="0.1524" layer="91"/>
+<wire x1="345.44" y1="246.38" x2="355.6" y2="246.38" width="0.1524" layer="91"/>
 <junction x="345.44" y="246.38"/>
-<wire x1="353.06" y1="246.38" x2="353.06" y2="241.3" width="0.1524" layer="91"/>
+<wire x1="355.6" y1="246.38" x2="355.6" y2="241.3" width="0.1524" layer="91"/>
 <pinref part="GND136" gate="1" pin="GND"/>
+<pinref part="LED5" gate="G$1" pin="C"/>
+<junction x="355.6" y="246.38"/>
+</segment>
+<segment>
+<pinref part="X1" gate="-3" pin="S"/>
+<wire x1="114.3" y1="259.08" x2="104.14" y2="259.08" width="0.1524" layer="91"/>
+<wire x1="104.14" y1="259.08" x2="104.14" y2="256.54" width="0.1524" layer="91"/>
+<pinref part="GND150" gate="1" pin="GND"/>
 </segment>
 </net>
@@
 </segment>
 </net>
+<net name="N$6" class="0">
+<segment>
+<pinref part="LED5" gate="G$1" pin="A"/>
+<pinref part="R11" gate="G$1" pin="1"/>
+<wire x1="355.6" y1="254" x2="355.6" y2="259.08" width="0.1524" layer="91"/>
+</segment>
+</net>
+<net name="HEARTBEAT" class="0">
+<segment>
+<pinref part="R11" gate="G$1" pin="2"/>
+<wire x1="355.6" y1="269.24" x2="355.6" y2="279.4" width="0.1524" layer="91"/>
+<label x="355.6" y="279.4" size="1.778" layer="95" rot="R90"/>
+</segment>
+<segment>
+<pinref part="SV1" gate="G$1" pin="3"/>
+<wire x1="5.08" y1="236.22" x2="-2.54" y2="236.22" width="0.1524" layer="91"/>
+<label x="-17.78" y="236.22" size="1.778" layer="95"/>
+</segment>
+</net>

Commit message: now using polarized symbol for tantalum caps
Parts:
- removed C104, C105, C106, C108, C110, C112, C115, C118, C138, C139, C140, C142, C144, C146, C149, C152, C34, C37, C65, C68: 10uF, rcl:C-EUC1206
- added C1, C10, C2, C21, C22, C23, C24, C25, C26, C27, C28, C29, C3, C30, C4, C5, C6, C7, C8, C9: 10uF, resistor:CPOL-EUSMCA
Connections:
- net ADC_1_VREF: now also C28.+; no longer C37.1
- net ADC_2_VREF: now also C30.+; no longer C68.1
- net DVCC: now also C1.+, C2.+, C21.+, C22.+; no longer C104.1, C105.1, C138.1, C139.1
- net GND: now also C1.-, C10.-, C2.-, C21.-, C22.-, C23.-, C24.-, C25.+, C26.+, C27.-, C28.-, C29.-, C3.-, C30.-, C4.-, C5.-, C6.-, C7.+, C8.+, C9.-; no longer C104.2, C105.2, C106.2, C108.2, C110.2, C112.2, C115.2, C118.2, C138.2, C139.2, C140.2, C142.2, C144.2, C146.2, C149.2, C152.2, C34.2, C37.2, C65.2, C68.2
- net VDD: now also C23.+, C24.+, C27.+, C29.+, C3.+, C5.+, C6.+, C9.+; no longer C106.1, C108.1, C115.1, C140.1, C142.1, C149.1, C34.1, C65.1
- net VREF_1: now also C4.+; no longer C118.1
- net VREF_2: now also C10.+; no longer C152.1
- net VSS: now also C25.-, C26.-, C7.-, C8.-; no longer C110.1, C112.1, C144.1, C146.1

Commit message: minor changes
Changed lines of the file:
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@@
 <?xml version="1.0" encoding="utf-8"?>
 <!DOCTYPE eagle SYSTEM "eagle.dtd">
-<eagle version="8.6.2">
+<eagle version="8.7.1">
 <drawing>
 <settings>
@@
 <part name="GND107" library="supply1" deviceset="GND" device=""/>
 <part name="GND108" library="supply1" deviceset="GND" device=""/>
-<part name="S1" library="1MS1T1B1M2QES-5" deviceset="1MS1T1B1M2QES-5" device=""/>
+<part name="S1" library="1MS1T1B1M2QES-5" deviceset="1MS1T1B1M2QES-5" device="" value=""/>
 <part name="GND135" library="supply1" library_urn="urn:adsk.eagle:library:371" deviceset="GND" device=""/>
 <part name="LED3" library="led" library_urn="urn:adsk.eagle:library:259" deviceset="TLLG4400" device="" package3d_urn="urn:adsk.eagle:package:15797/1" value=""/>
